Commit message: Rebuild the description from the CAD, shared with a MuJoCo model
Export one mesh per part from the STEP assemblies with export_step_meshes.py
and export_torso.py, and use the same meshes, kinematics and inertial data in
the URDF and in mujoco/mobile_platform.xml. The two agree to 0.000 mm on every
drive and wheel frame, and both come to 94.83 kg.

Fix two errors in the drive units. The pivot sat on the wheel axle, 10 mm
inboard of the slew bearing, leaving no castor offset for the wheel pair to
steer with; and the attachment origins had x and y swapped, which put the four
units on a rectangle turned 90 degrees from the real one. The wheel's polar
moment now sits on its spin axis.

Add the torso, up to the arm mounting plates, placed from the full-assembly
STEP, and display_eddie_base.launch.py for the base on its own. Drop eddie_urdf
and the meshes it duplicated.

File: urdf/eddie_base.macro.xacro (robot description, xacro)
@@ -6,31 +6,26 @@
         <!-- Properties -->
         <xacro:property name="mesh_package" value="eddie_description" />
-        <xacro:property name="eddie_base_file" value="kelo_base.stl" />
-        <xacro:property name="eddie_torso_file" value="kelo_torso.stl" />
-        <!-- wheel unit attachments -->
+        <!-- The CAD meshes are y-up and in millimetres. -->
+        <xacro:property name="mesh_rpy" value="1.5708 0 1.5708" />
+        <xacro:property name="mesh_scale" value="0.001 0.001 0.001" />
+        <!-- wheel unit attachments, on the units' slew-bearing axes -->
         <xacro:property name="front_left_attachment_origin">
-            <origin xyz="0.2078 0.1880 -0.0632" rpy="0 0 1.5708" />
+            <origin xyz="0.18813 0.20748 -0.1273" rpy="0 0 0" />
         </xacro:property>
         <xacro:property name="rear_left_attachment_origin">
-            <origin xyz="-0.2078 0.1880 -0.0632" rpy="0 0 1.5708" />
+            <origin xyz="-0.18787 0.20748 -0.1273" rpy="0 0 0" />
         </xacro:property>
         <xacro:property name="rear_right_attachment_origin">
-            <origin xyz="-0.2078 -0.1880 -0.0632" rpy="0 0 -1.5708" />
+            <origin xyz="-0.18787 -0.20752 -0.1273" rpy="0 0 0" />
         </xacro:property>
         <xacro:property name="front_right_attachment_origin">
-            <origin xyz="0.2078 -0.1880 -0.0632" rpy="0 0 -1.5708" />
-        </xacro:property>
-        <xacro:property name="front_right_struct_wrt_attachment_rpy" value="0 0 -1.5708" />
-        <xacro:property name="front_left_struct_wrt_attachment_rpy" value="0 0 1.5708" />
-        <xacro:property name="rear_right_struct_wrt_attachment_rpy" value="0 0 -1.5708" />
-        <xacro:property name="rear_left_struct_wrt_attachment_rpy" value="0 0 1.5708" />
+            <origin xyz="0.18813 -0.20752 -0.1273" rpy="0 0 0" />
+        </xacro:property>
         <!-- base link origin -->
         <xacro:property name="base_link_origin">
             <origin xyz="0 0 0.2164" rpy="0 0 0" />
         </xacro:property>
-        <!-- torso origin -->
-        <xacro:property name="torso_origin_wrt_base_link">
-            <origin xyz="-0.1738 0.0003 0.4184" rpy="0 0 1.5708" />
-        </xacro:property>
+        <!-- torso origin, from "Full assembly Robot 7_5D.STEP" -->
+        <xacro:property name="torso_xyz" value="-0.1738 0.0003 0.4184" />
         <!-- arm attachment origins -->
         <xacro:property name="left_arm_attachment_origin">
@@ -49,27 +44,57 @@
             <!-- base -->
             <visual>
-                <origin rpy="0 0 0" xyz="0 0 0" />
-                <geometry>
-                    <mesh filename="package://${mesh_package}/meshes/${eddie_base_file}" />
-                </geometry>
-                <material name="light_gray" />
-            </visual>
+                <origin rpy="${mesh_rpy}" xyz="0 0 0" />
+                <geometry>
+                    <mesh filename="package://${mesh_package}/meshes/casing.stl" scale="${mesh_scale}" />
+                </geometry>
+                <material name="casing_grey" />
+            </visual>
+            <visual>
+                <origin rpy="${mesh_rpy}" xyz="0 0 0" />
+                <geometry>
+                    <mesh filename="package://${mesh_package}/meshes/panel.stl" scale="${mesh_scale}" />
+                </geometry>
+                <material name="casing_grey" />
+            </visual>
+            <visual>
+                <origin rpy="${mesh_rpy}" xyz="0 0 0" />
+                <geometry>
+                    <mesh filename="package://${mesh_package}/meshes/cover.stl" scale="${mesh_scale}" />
+                </geometry>
+                <material name="cover_light" />
+            </visual>
+            <visual>
+                <origin rpy="${mesh_rpy}" xyz="0 0 0" />
+                <geometry>
+                    <mesh filename="package://${mesh_package}/meshes/lidar.stl" scale="${mesh_scale}" />
+                </geometry>
+                <material name="lidar_grey" />
+            </visual>
+            <!-- only the outer shell can hit the world -->
             <collision>
-                <geometry>
-                    <mesh filename="package://${mesh_package}/meshes/${eddie_base_file}" />
+                <origin rpy="${mesh_rpy}" xyz="0 0 0" />
+                <geometry>
+                    <mesh filename="package://${mesh_package}/meshes/casing.stl" scale="${mesh_scale}" />
                 </geometry>
             </collision>
             <!-- torso -->
             <visual>
-                <xacro:insert_block name="torso_origin_wrt_base_link" />
-                <geometry>
-                    <mesh filename="package://${mesh_package}/meshes/${eddie_torso_file}" />
-                </geometry>
-                <material name="metallic_silver" />
+                <origin rpy="${mesh_rpy}" xyz="${torso_xyz}" />
+                <geometry>
+                    <mesh filename="package://${mesh_package}/meshes/torso.stl" scale="${mesh_scale}" />
+                </geometry>
+                <material name="cover_light" />
+            </visual>
+            <visual>
+                <origin rpy="${mesh_rpy}" xyz="${torso_xyz}" />
+                <geometry>
+                    <mesh filename="package://${mesh_package}/meshes/torso_mounts.stl" scale="${mesh_scale}" />
+                </geometry>
+                <material name="mount_grey" />
             </visual>
             <collision>
-                <xacro:insert_block name="torso_origin_wrt_base_link" />
-                <geometry>
-                    <mesh filename="package://${mesh_package}/meshes/${eddie_torso_file}" />
+                <origin rpy="${mesh_rpy}" xyz="${torso_xyz}" />
+                <geometry>
+                    <mesh filename="package://${mesh_package}/meshes/torso.stl" scale="${mesh_scale}" />
                 </geometry>
             </collision>
@@ -158,5 +183,5 @@
             use_kelo_tulip="${use_kelo_tulip}"
             struct_prefix="${robot_prefix}front_left_drive_"
-            struct_wrt_attachment_rpy="${front_left_struct_wrt_attachment_rpy}">
+            mirrored="true">
             <xacro:insert_block name="front_left_attachment_origin" />
         </xacro:kelo_drive_unit>
@@ -168,5 +193,5 @@
             use_kelo_tulip="${use_kelo_tulip}"
             struct_prefix="${robot_prefix}rear_left_drive_"
-            struct_wrt_attachment_rpy="${rear_left_struct_wrt_attachment_rpy}">
+            mirrored="true">
             <xacro:insert_block name="rear_left_attachment_origin" />
         </xacro:kelo_drive_unit>
@@ -178,5 +203,5 @@
             use_kelo_tulip="${use_kelo_tulip}"
             struct_prefix="${robot_prefix}rear_right_drive_"
-            struct_wrt_attachment_rpy="${front_right_struct_wrt_attachment_rpy}">
+            mirrored="false">
             <xacro:insert_block name="rear_right_attachment_origin" />
         </xacro:kelo_drive_unit>
@@ -188,5 +213,5 @@
             use_kelo_tulip="${use_kelo_tulip}"
             struct_prefix="${robot_prefix}front_right_drive_"
-            struct_wrt_attachment_rpy="${rear_right_struct_wrt_attachment_rpy}">
+            mirrored="false">
             <xacro:insert_block name="front_right_attachment_origin" />
         </xacro:kelo_drive_unit>

File: urdf/kelo_drive_unit.macro.xacro (robot description, xacro)
@@ -3,7 +3,9 @@
     <!-- Include macro files -->
     <xacro:include filename="$(find eddie_description)/urdf/kelo_hub_wheel.macro.xacro" />
+    <!-- The pivot is the unit's slew-bearing axis; the 10.1 mm castor offset that
+         lets the wheel pair steer it sits in the wheel origins, not the pivot. -->
     <xacro:macro name="kelo_drive_unit"
-        params="parent use_ros2_control use_gz_sim use_kelo_tulip struct_prefix *attachment_origin
-    struct_wrt_attachment_rpy">
+        params="parent use_ros2_control use_gz_sim use_kelo_tulip struct_prefix
+    mirrored:=false *attachment_origin">
         <!-- pivot joint type based on use_kelo_tulip -->
         <xacro:if value="${use_kelo_tulip}">
@@ -15,29 +17,17 @@
         <!-- Properties -->
         <xacro:property name="mesh_package" value="eddie_description" />
-        <xacro:property name="struct_mesh_file" value="kelo_drive.stl" />
-        <xacro:property name="struct_attachment_mesh_file" value="kelo_drive_attachments.stl" />
-        <!-- struct -->
-        <xacro:property name="struct_wrt_attachment_origin">
-            <origin xyz="-0.0100 -0.0006 -0.0641" rpy="${struct_wrt_attachment_rpy}" />
-        </xacro:property>
+        <xacro:property name="struct_mesh_file" value="drive.stl" />
+        <!-- The mirrored units are the same part half a turn about the pivot. -->
+        <xacro:if value="${mirrored}">
+            <xacro:property name="mesh_rpy" value="1.5708 0 -1.5708" />
+            <xacro:property name="flip" value="-1" />
+        </xacro:if>
+        <xacro:unless value="${mirrored}">
+            <xacro:property name="mesh_rpy" value="1.5708 0 1.5708" />
+            <xacro:property name="flip" value="1" />
+        </xacro:unless>
         <!-- Links -->
-        <link name="${struct_prefix}attachment_link">
-            <visual>
-                <origin rpy="0 0 0" xyz="0 0 0" />
-                <geometry>
-                    <mesh filename="package://${mesh_package}/meshes/${struct_attachment_mesh_file}" />
-                </geometry>
-                <material name="metallic_silver" />
-            </visual>
-            <collision>
-                <geometry>
-                    <mesh filename="package://${mesh_package}/meshes/${struct_attachment_mesh_file}" />
-                </geometry>
-            </collision>
-            <inertial>
-                <mass value="0.5" />
-                <inertia ixx="0.00042" ixy="0" ixz="0" iyy="0.00042" iyz="0" izz="0.0008" />
-            </inertial>
-        </link>
+        <!-- massless: a frame; the unit's mass is on the part that turns -->
+        <link name="${struct_prefix}attachment_link" />
         <!-- attachment joint -->
         <joint name="${struct_prefix}attachment_joint" type="fixed">
@@ -48,18 +38,13 @@
         <link name="${struct_prefix}struct_link">
             <visual>
-                <origin rpy="0 0 0" xyz="0 0 0" />
+                <origin rpy="${mesh_rpy}" xyz="0 0 0" />
                 <geometry>
-                    <mesh filename="package://${mesh_package}/meshes/${struct_mesh_file}" />
+                    <mesh filename="package://${mesh_package}/meshes/${struct_mesh_file}" scale="0.001 0.001 0.001" />
                 </geometry>
-                <material name="metallic_silver" />
+                <material name="drive_grey" />
             </visual>
-            <collision>
-                <geometry>
-                    <mesh filename="package://${mesh_package}/meshes/${struct_mesh_file}" />
-                </geometry>
-            </collision>
             <inertial>
                 <mass value="1.392" />
-                <origin xyz="0 0 0.006" rpy="0 0 0" />
+                <origin xyz="0 ${flip * 0.0101} 0" rpy="0 0 0" />
                 <inertia ixx="0.004574163" ixy="0" ixz="0" iyy="0.004344228" iyz="0"
                     izz="0.004640438" />
@@ -70,5 +55,5 @@
             <parent link="${struct_prefix}attachment_link" />
             <child link="${struct_prefix}struct_link" />
-            <xacro:insert_block name="struct_wrt_attachment_origin" />
+            <origin xyz="0 0 0" rpy="0 0 0" />
             <axis xyz="0 0 1" />
             <dynamics damping="0.1" friction="0.1" />
@@ -96,8 +81,11 @@
         <xacro:property name="right_wheel_prefix" value="r_wheel_" />
         <xacro:property name="right_wheel_origin">
-            <origin xyz="0.0008 0.0407 -0.0366" rpy="-1.5708 0 0" />
+            <origin xyz="${flip * -0.040500} ${flip * 0.010108} -0.036587" rpy="0 0 0" />
         </xacro:property>
         <xacro:kelo_hub_wheel wheel_prefix="${struct_prefix}${right_wheel_prefix}"
             parent="${struct_prefix}struct_link"
+            wheel_mesh="wheel_a.stl"
+            tyre_mesh="tyre_a.stl"
+            mesh_rpy="${mesh_rpy}"
             use_ros2_control="${use_ros2_control}"
             use_gz_sim="${use_gz_sim}"
@@ -108,8 +96,11 @@
         <xacro:property name="left_wheel_prefix" value="l_wheel_" />
         <xacro:property name="left_wheel_origin">
-            <origin xyz="0.0008 -0.0403 -0.0366" rpy="1.5708 3.1416 0" />
+            <origin xyz="${flip * 0.040500} ${flip * 0.009890} -0.036587" rpy="0 0 0" />
         </xacro:property>
         <xacro:kelo_hub_wheel wheel_prefix="${struct_prefix}${left_wheel_prefix}"
             parent="${struct_prefix}struct_link"
+            wheel_mesh="wheel_b.stl"
+            tyre_mesh="tyre_b.stl"
+            mesh_rpy="${mesh_rpy}"
             use_ros2_control="${use_ros2_control}"
             use_gz_sim="${use_gz_sim}"

File: urdf/kelo_hub_wheel.macro.xacro (robot description, xacro)
@@ -2,8 +2,7 @@
 <robot xmlns:xacro="http://www.ros.org/wiki/xacro" name="kelo_hub_wheel">
     <xacro:macro name="kelo_hub_wheel"
-        params="wheel_prefix parent *wheel_origin use_ros2_control use_gz_sim use_kelo_tulip">
-        <!-- Properties -->
+        params="wheel_prefix parent *wheel_origin wheel_mesh tyre_mesh mesh_rpy
+    use_ros2_control use_gz_sim use_kelo_tulip">
         <xacro:property name="mesh_package" value="eddie_description" />
-        <xacro:property name="wheel_mesh_file" value="hub_wheel.stl" />
         <!-- wheel joint type based on use_kelo_tulip -->
         <xacro:if value="${use_kelo_tulip}">
@@ -16,13 +15,22 @@
         <link name="${wheel_prefix}link">
             <visual>
-                <origin rpy="0 0 0" xyz="0 0 0" />
+                <origin rpy="${mesh_rpy}" xyz="0 0 0" />
                 <geometry>
-                    <mesh filename="package://${mesh_package}/meshes/${wheel_mesh_file}" />
+                    <mesh filename="package://${mesh_package}/meshes/${wheel_mesh}" scale="0.001 0.001 0.001" />
                 </geometry>
-                <material name="almost_black" />
+                <material name="wheel_light" />
             </visual>
+            <visual>
+                <origin rpy="${mesh_rpy}" xyz="0 0 0" />
+                <geometry>
+                    <mesh filename="package://${mesh_package}/meshes/${tyre_mesh}" scale="0.001 0.001 0.001" />
+                </geometry>
+                <material name="tyre_dark" />
+            </visual>
+            <!-- only the tread ring touches the ground -->
             <collision>
+                <origin rpy="${mesh_rpy}" xyz="0 0 0" />
                 <geometry>
-                    <mesh filename="package://${mesh_package}/meshes/${wheel_mesh_file}" />
+                    <mesh filename="package://${mesh_package}/meshes/${tyre_mesh}" scale="0.001 0.001 0.001" />
                 </geometry>
             </collision>
@@ -35,9 +43,10 @@
                 </friction>
             </surface>
+            <!-- spin axis is x, so the polar moment is ixx -->
             <inertial>
                 <mass value="1.563" />
-                <origin rpy="0 0 0" xyz="0 0.00003 -0.00044" />
-                <inertia ixx="0.001012837" ixy="0" ixz="0" iyy="0.001013130" iyz="0"
-                    izz="0.001579986" />
+                <origin rpy="0 0 0" xyz="0 0 0" />
+                <inertia ixx="0.001579986" ixy="0" ixz="0" iyy="0.001012837" iyz="0"
+                    izz="0.001013130" />
             </inertial>
         </link>
@@ -47,5 +56,5 @@
             <child link="${wheel_prefix}link" />
             <xacro:insert_block name="wheel_origin" />
-            <axis xyz="0 0 1" />
+            <axis xyz="-1 0 0" />
             <dynamics damping="0.1" friction="0.1" />
         </joint>

File: urdf/materials.xacro (robot description, xacro)
@@ -1,4 +1,27 @@
 <?xml version="1.0"?>
 <robot xmlns:xacro="http://www.ros.org/wiki/xacro" name="eddie_materials">
+    <!-- Part colours, from meshes/colors.json and meshes/torso_colors.json. -->
+    <material name="casing_grey">
+        <color rgba="0.25 0.25 0.26 1.0" />
+    </material>
+    <material name="cover_light">
+        <color rgba="0.898 0.918 0.929 1.0" />
+    </material>
+    <material name="lidar_grey">
+        <color rgba="0.792 0.82 0.933 1.0" />
+    </material>
+    <material name="mount_grey">
+        <color rgba="0.42 0.42 0.43 1.0" />
+    </material>
+    <material name="drive_grey">
+        <color rgba="0.35 0.35 0.35 1.0" />
+    </material>
+    <material name="wheel_light">
+        <color rgba="0.996 0.996 1.0 1.0" />
+    </material>
+    <material name="tyre_dark">
+        <color rgba="0.251 0.251 0.251 1.0" />
+    </material>
+    <!-- referenced by the arm and gripper descriptions -->
     <material name="metallic_silver">
         <color rgba="0.5 0.5 0.5 1.0" />
